File: HW/KiCad/ATmega2560-MegaPro-001/ATmega2560-MegaPro-001.kicad_pcb (KiCad board)
At the start: 2 copper layers, 55.9 x 40.8 mm, 50 parts, among them J1 Conn_02x16_Odd_Even, J2 Conn_02x21_Odd_Even, J3 Conn_02x03_Odd_Even, J4 AVR-ISP-6, J5 USB_B_Micro, U1 ATMEGA2560-16AU, U2 CH340G, U3 AMS1117-5.0, U4 AMS1117-3.3, Y1 16 MHz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

Commit message: +3d models, +Pins.rst, some reorganisation
Parts:
- R12: value R -> 102
Changed lines of the file:
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@@
 			)
 		)
-		(property "Value" "R"
+		(property "Value" "102"
 			(at 0 0.0076 0)
 			(layer "F.Fab")
