File: HW/KiCad/MHF-001/MHF-001.kicad_sch (KiCad schematic)
At the start: 219 parts, among them J1 DE15_Socket_HighDensity_Mount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, J10 I2C, J11 POWER, J2 Mini-DIN-6, J3 Conn_Coaxial, J4 Conn_02x32_Odd_Even, J5 USB_B_Micro, J6 02x32, J7 SPI, J8 AVR-ISP-6, J9 Serial, M3 CY7C109D-10ZXI, M5 CY7C109D-10ZXI, Q1 BC107, U1 ATMEGA2560-16AU, U10 74HC245, U11 74HC245, U12 74HC245, U13 CH340G, U14 AMS1117-5.0, U15 AMS1117-3.3, U2 74HC14, U3 74LS08, U4 74HC165, U6 74AHC373PW, U7 74HC595, U8 74HC595, U9 74HC157, Y1 16 MHz, Y2 12 MHz

Commit message: saved lot of pins by removing unnecessery/redundant signals
Parts:
- removed JP101, JP108, JP93, JP96, JP97: SolderJumper_3_Open, Jumper:SolderJumper-3_P1.3mm_Open_RoundedPad1.0x1.5mm, symbol Jumper:SolderJumper_3_Open
Connections:
- net A_BUS is gone; now on net A_HALT: J4.29 (Pin_29), J6.29 (Pin_29)
- net A_SHARE_BUSY is gone; now on net A_SHARE_REQUEST: J4.37 (Pin_37), J6.37 (Pin_37)
- net A_SHARE_WANTED is gone; now on net A_G_D_DIR: J4.45 (Pin_45), J6.45 (Pin_45)
- net A_WRITE is gone; now on net A_SHARE_GRANTED: J4.35 (Pin_35), J6.35 (Pin_35)
- net B_BUS is gone; now on net B_HALT: J4.30 (Pin_30), J6.30 (Pin_30)
- net B_SHARE_BUSY is gone; now on net B_SHARE_REQUEST: J4.38 (Pin_38), J6.38 (Pin_38)
- net B_SHARE_WANTED is gone; now on net B_G_D_DIR: J4.46 (Pin_46), J6.46 (Pin_46)
- net B_WRITE is gone; now on net B_SHARE_GRANTED: J4.36 (Pin_36), J6.36 (Pin_36)
- net G_D_OE is gone; now on net G_ENABLE: JP106.2 (C), U10.19 (CE)
- net X_SHARE_BUSY is gone; now on net X_SHARE_GRANTED: JP29.2 (B)
- net X_WRITE is gone; now on net X_READ: JP28.2 (B)
- net A_G_A_DIR: now also J4.47 (Pin_47), J6.47 (Pin_47); no longer J4.57 (Pin_57), J6.57 (Pin_57)
- net A_G_D_DIR: no longer J4.53 (Pin_53), J6.53 (Pin_53)
- net A_HALT: no longer J4.31 (Pin_31), J6.31 (Pin_31)
- net A_READ: now also J4.31 (Pin_31), J6.31 (Pin_31); no longer J4.33 (Pin_33), J6.33 (Pin_33)
- net A_SHARE_DIRTY: now also J4.33 (Pin_33), J6.33 (Pin_33); no longer J4.39 (Pin_39), J6.39 (Pin_39)
- net A_SHARE_GRANTED: no longer J4.41 (Pin_41), J6.41 (Pin_41)
- net A_SHARE_REQUEST: no longer J4.43 (Pin_43), J6.43 (Pin_43)
- net A_S_ENABLE: now also J4.39 (Pin_39), J6.39 (Pin_39); no longer J4.47 (Pin_47), J6.47 (Pin_47)
- net A_S_READ: now also J4.41 (Pin_41), J6.41 (Pin_41); no longer J4.49 (Pin_49), J6.49 (Pin_49)
- net A_S_WRITE: now also J4.43 (Pin_43), J6.43 (Pin_43); no longer J4.51 (Pin_51), J6.51 (Pin_51)
- net B_G_A_DIR: now also J4.48 (Pin_48), J6.48 (Pin_48); no longer J4.58 (Pin_58), J6.58 (Pin_58)
- net B_G_D_DIR: no longer J4.54 (Pin_54), J6.54 (Pin_54)
- net B_HALT: no longer J4.32 (Pin_32), J6.32 (Pin_32)
- net B_READ: now also J4.32 (Pin_32), J6.32 (Pin_32); no longer J4.34 (Pin_34), J6.34 (Pin_34)
- net B_SHARE_DIRTY: now also J4.34 (Pin_34), J6.34 (Pin_34); no longer J4.40 (Pin_40), J6.40 (Pin_40)
- net B_SHARE_GRANTED: no longer J4.42 (Pin_42), J6.42 (Pin_42)
- net B_SHARE_REQUEST: no longer J4.44 (Pin_44), J6.44 (Pin_44)
- net B_S_ENABLE: now also J4.40 (Pin_40), J6.40 (Pin_40); no longer J4.48 (Pin_48), J6.48 (Pin_48)
- net B_S_READ: now also J4.42 (Pin_42), J6.42 (Pin_42); no longer J4.50 (Pin_50), J6.50 (Pin_50)
- net B_S_WRITE: now also J4.44 (Pin_44), J6.44 (Pin_44); no longer J4.52 (Pin_52), J6.52 (Pin_52)
- net X_HALT: now also JP27.2 (B); no longer JP53.2 (B)
- net X_READ: no longer JP27.2 (B)
- net X_SHARE_DIRTY: now also JP31.2 (B); no longer JP30.2 (B)
- net X_SHARE_GRANTED: no longer JP31.2 (B)
- net X_SHARE_REQUEST: now also JP30.2 (B); no longer JP32.2 (B)
- net A_G_A_OE: no longer names the net of J6.59 (Pin_59)
- net A_G_A_OE: no longer J4.59 (Pin_59)
- removed net A_G_D_OE: J4.55 (Pin_55), J6.55 (Pin_55), JP106.1 (A)
- net B_G_A_OE: no longer names the net of J6.60 (Pin_60)
- net B_G_A_OE: no longer J4.60 (Pin_60)
- removed net B_G_D_OE: J4.56 (Pin_56), J6.56 (Pin_56), JP106.3 (B)
- net G_A_OE renamed G_ENABLE
- net X_BUS: no longer names the net of JP54.2 (B)
- net X_SHARE_WANTED: no longer names the net of JP38.2 (B)
- new net A_G_ENABLE: J4.49 (Pin_49), J6.49 (Pin_49), JP106.1 (A)
- new net B_G_ENABLE: J4.50 (Pin_50), J6.50 (Pin_50), JP106.3 (B)
- no-connect marks 26 -> 54
Other:
- note added: "EMS RAM 8000-9FFF A000-BFFFF (shared between Arduino and HD6309)"
- note removed: "RAM Midlle 8000-9FFF (shared with Arduino)"

Commit message: +NetJoint
Parts:
- added J12: Reset, Connector_Wire:SolderWire-0.5sqmm_1x01_D0.9mm_OD2.1mm, symbol Connector_Generic:Conn_01x01
- added J13: AREF, Connector_Wire:SolderWire-0.5sqmm_1x01_D0.9mm_OD2.1mm, symbol Connector_Generic:Conn_01x01
- added J14: XTAL2, Connector_Wire:SolderWire-0.5sqmm_1x01_D0.9mm_OD2.1mm, symbol Connector_Generic:Conn_01x01
- added J15: XTAL1, Connector_Wire:SolderWire-0.5sqmm_1x01_D0.9mm_OD2.1mm, symbol Connector_Generic:Conn_01x01
- added J16: AVCC, Connector_Wire:SolderWire-0.5sqmm_1x01_D0.9mm_OD2.1mm, symbol Connector_Generic:Conn_01x01
- added JP93: SolderJumper_2_Bridged, Jumper:SolderJumper-2_P1.3mm_Bridged_Pad1.0x1.5mm, symbol Jumper:SolderJumper_2_Bridged
- added N1, N2, N3, N4: ~, Gilhad:NetJoint, symbol PCM_Gilhad_symbols:NetJoint
- R32, R33: footprint Resistor_SMD:R_0603_1608Metric_Pad0.98x0.95mm_HandSolder -> Resistor_SMD:R_0805_2012Metric_Pad1.20x1.40mm_HandSolder
Connections:
- net +5V: now also J10.3 (Pin_3), JP93.1 (A); no longer J10.4 (Pin_4), U1.100 (AVCC)
- net AREF: now also J13.1 (Pin_1)
- net Bb: now also N2.2; no longer R5.1, U3.1
- net GND: now also J10.4 (Pin_4); no longer J10.3 (Pin_3)
- net Reset: now also J12.1 (Pin_1)
- net SCL: now also J10.1 (Pin_1); no longer J10.2 (Pin_2)
- net SDA: now also J10.2 (Pin_2); no longer J10.1 (Pin_1)
- net SYNC_RCA: now also N4.2; no longer JP85.2 (B), U4.3 (D4)
- net Shared_Address_A16: now also N1.1; no longer JP14.2 (B), JP92.2 (C)
- net VGA data 3: now also N3.1; no longer U3.2
- net XTAL1: now also J15.1 (Pin_1)
- net XTAL2: now also J14.1 (Pin_1)
- net X_HALT: now also JP38.2 (B); no longer JP27.2 (B)
- net X_READ: now also JP32.2 (B); no longer JP28.2 (B)
- new net: J16.1 (Pin_1), JP93.2 (B), U1.100 (AVCC)
- new net SIGNAL_RCA: JP28.2 (B), R5.1, U3.1
- new net VGA data 4: JP85.2 (B), N4.1, U4.3 (D4)
- new net X16: JP14.2 (B), JP92.2 (C), N1.2
- new net ~{SUPRESS}: N3.2, U3.2
- no-connect marks 54 -> 53
Other:
- note added: "RX for Signal_RCA"
- moved on the sheet: C5, J10, J7, J9

Commit message: cleaning
Parts:
- removed JP1, JP10, JP11, JP12, JP13, JP14, JP15, JP16, JP17, JP18, JP19, JP2, JP20, JP21, JP22, JP23, JP24, JP25, JP26, JP27, JP28, JP29, JP3, JP30, JP31, JP32, JP33, JP34, JP35, JP36, JP37, JP38, JP39, JP4, JP40, JP41, JP42, JP43, JP44, JP45, JP46, JP47, JP48, JP49, JP5, JP50, JP51, JP52, JP53, JP54, JP57, JP58, JP59, JP6, JP60, JP61, JP62, JP63, JP64, JP65, JP66, JP67, JP68, JP69, JP7, JP70, JP71, JP72, JP73, JP74, JP75, JP76, JP77, JP78, JP79, JP8, JP80, JP81, JP82, JP83, JP84, JP85, JP86, JP87, JP88, JP9: SolderJumper_2_Bridged, Jumper:SolderJumper-2_P1.3mm_Bridged_Pad1.0x1.5mm, symbol Jumper:SolderJumper_2_Bridged
- removed N1, N2: ~, Gilhad:NetJoint, symbol PCM_Gilhad_symbols:NetJoint
- added R40: 1k, Resistor_SMD:R_0603_1608Metric_Pad0.98x0.95mm_HandSolder, symbol Device:R
Connections:
- net PA0 is gone; now on net XAD0: PA1.1 (Pin_1), U1.78 ((AD0)PA0)
- net PA1 is gone; now on net XAD1: PA1.2 (Pin_2), U1.77 ((AD1)PA1)
- net PA2 is gone; now on net XAD2: PA1.3 (Pin_3), U1.76 ((AD2)PA2)
- net PA3 is gone; now on net XAD3: PA1.4 (Pin_4), U1.75 ((AD3)PA3)
- net PA4 is gone; now on net XAD4: PA1.5 (Pin_5), U1.74 ((AD4)PA4)
- net PA5 is gone; now on net XAD5: PA1.6 (Pin_6), U1.73 ((AD5)PA5)
- net PA6 is gone; now on net XAD6: PA1.7 (Pin_7), U1.72 ((AD6)PA6)
- net PA7 is gone; now on net XAD7: PA1.8 (Pin_8), U1.71 ((AD7)PA7)
- net PB0 is gone; now on net SS: PB1.1 (Pin_1), U1.19 ((SS/PCINT0)PB0)
- net PB1 is gone; now on net SCK: PB1.2 (Pin_2), U1.20 ((SCK/PCINT1)PB1)
- net PB2 is gone; now on net MOSI: PB1.3 (Pin_3), U1.21 ((MOSI/PCINT2)PB2)
- net PB3 is gone; now on net MISO: PB1.4 (Pin_4), U1.22 ((MISO/PCINT3)PB3)
- net PB4 is gone; now on net PS2-OE: PB1.5 (Pin_5), U1.23 ((OC2A/PCINT4)PB4)
- net PB5 is gone; now on net X16: PB1.6 (Pin_6), U1.24 ((OC1A/PCINT5)PB5)
- net PB6 is gone; now on net HSyncVGA: PB1.7 (Pin_7), U1.25 ((OC1B/PCINT6)PB6)
- net PB7 is gone; now on net VGA Latch: PB1.8 (Pin_8), U1.26 ((OC0A/OC1C/PCINT7)PB7)
- net PC0 is gone; now on net XAA0: PC1.1 (Pin_1), U1.53 ((A8)PC0)
- net PC1 is gone; now on net XAA1: PC1.2 (Pin_2), U1.54 ((A9)PC1)
- net PC2 is gone; now on net XAA2: PC1.3 (Pin_3), U1.55 ((A10)PC2)
- net PC3 is gone; now on net XAA3: PC1.4 (Pin_4), U1.56 ((A11)PC3)
- net PC4 is gone; now on net XAA4: PC1.5 (Pin_5), U1.57 ((A12)PC4)
- net PC5 is gone; now on net XAA5: PC1.6 (Pin_6), U1.58 ((A13)PC5)
- net PC6 is gone; now on net XAA6: PC1.7 (Pin_7), U1.59 ((A14)PC6)
- net PC7 is gone; now on net XAA7: PC1.8 (Pin_8), U1.60 ((A15)PC7)
- net PD0 is gone; now on net SCL: PD1.1 (Pin_1), R33.2, U1.43 ((SCL/INT0)PD0)
- net PD1 is gone; now on net SDA: PD1.2 (Pin_2), R32.2, U1.44 ((SDA/INT1)PD1)
- net PD3 is gone; now on net SIGNAL_RCA: PD1.4 (Pin_4), U1.46 ((TXD1/INT3)PD3)
- net PD4 is gone; now on net X_SHARE_GRANTED: PD1.5 (Pin_5), U1.47 ((ICP1)PD4)
- net PD5 is gone; now on net X_SHARE_REQUEST: PD1.6 (Pin_6), U1.48 ((XCK1)PD5)
- net PD6 is gone; now on net X_SHARE_DIRTY: PD1.7 (Pin_7), U1.49 ((T1)PD6)
- net PD7 is gone; now on net X_READ: PD1.8 (Pin_8), U1.50 ((T0)PD7)
- net PE0 is gone; now on net TX: PE1.1 (Pin_1), U1.2 ((RXD0/PCIN8)PE0)
- net PE1 is gone; now on net RX: PE1.2 (Pin_2), U1.3 ((TXD0)PE1)
- net PE2 is gone; now on net CTS: PE1.3 (Pin_3), U1.4 ((XCK0/AIN0)PE2)
- net PE3 is gone; now on net RTS: PE1.4 (Pin_4), U1.5 ((OC3A/AIN1)PE3)
- net PE4 is gone; now on net VSyncVGA: PE1.5 (Pin_5), U1.6 ((OC3B/INT4)PE4)
- net PE5 is gone; now on net X_HALT: PE1.6 (Pin_6), U1.7 ((OC3C/INT5)PE5)
- net PE6 is gone; now on net Inside: PE1.7 (Pin_7), U1.8 ((T3/INT6)PE6)
- net PE7 is gone; now on net 16MHz: PE1.8 (Pin_8), U1.9 ((CLKO/ICP3/INT7)PE7)
- net PF0 is gone; now on net Shared_data_D0: PF1.1 (Pin_1), U1.97 ((ADC0)PF0)
- net PF1 is gone; now on net Shared_data_D1: PF1.2 (Pin_2), U1.96 ((ADC1)PF1)
- net PF2 is gone; now on net Shared_data_D2: PF1.3 (Pin_3), U1.95 ((ADC2)PF2)
- net PF3 is gone; now on net Shared_data_D3: PF1.4 (Pin_4), U1.94 ((ADC3)PF3)
- net PF4 is gone; now on net Shared_data_D4: PF1.5 (Pin_5), U1.93 ((ADC4/TCK)PF4)
- net PF5 is gone; now on net Shared_data_D5: PF1.6 (Pin_6), U1.92 ((ADC5/TMS)PF5)
- net PF6 is gone; now on net Shared_data_D6: PF1.7 (Pin_7), U1.91 ((ADC6/TDO)PF6)
- net PF7 is gone; now on net Shared_data_D7: PF1.8 (Pin_8), U1.90 ((ADC7/TDI)PF7)
- net PG0 is gone; now on net WE: PG1.1 (Pin_1), U1.51 ((WR)PG0)
- net PG1 is gone; now on net RD: PG1.2 (Pin_2), U1.52 ((RD)PG1)
- net PG2 is gone; now on net ALE: PG1.3 (Pin_3), U1.70 ((ALE)PG2)
- net PG3 is gone; now on net XAA16: PG1.4 (Pin_4), U1.28 ((TOSC2)PG3)
- net PH0 is gone; now on net Ib: PH1.1 (Pin_1), U1.12 (PH0(RXD2))
- net PH1 is gone; now on net Bb: PH1.2 (Pin_2), U1.13 (PH1(TXD2))
- net PH2 is gone; now on net Gb: PH1.3 (Pin_3), U1.14 (PH2(XCK2))
- net PH3 is gone; now on net Rb: PH1.4 (Pin_4), U1.15 (PH3(OC4A))
- net PH4 is gone; now on net If: PH1.5 (Pin_5), U1.16 (PH4(OC4B))
- net PH5 is gone; now on net Bf: PH1.6 (Pin_6), U1.17 (PH5(OC4C))
- net PH6 is gone; now on net Gf: PH1.7 (Pin_7), U1.18 (PH6(OC2B))
- net PH7 is gone; now on net Rf: PH1.8 (Pin_8), U1.27 (PH7(T4))
- net PJ0 is gone; now on net Shared_Address_A0: PJ1.1 (Pin_1), U1.63 (PJ0(RXD3/PCINT9))
- net PJ1 is gone; now on net Shared_Address_A1: PJ1.2 (Pin_2), U1.64 (PJ1(TXD3/PCINT10))
- net PJ2 is gone; now on net Shared_Address_A2: PJ1.3 (Pin_3), U1.65 (PJ2(XCK3/PCINT11))
- net PJ3 is gone; now on net Shared_Address_A3: PJ1.4 (Pin_4), U1.66 (PJ3(PCINT12))
- net PJ4 is gone; now on net Shared_Address_A4: PJ1.5 (Pin_5), U1.67 (PJ4(PCINT13))
- net PJ5 is gone; now on net Shared_Address_A5: PJ1.6 (Pin_6), U1.68 (PJ5(PCINT14))
- net PJ6 is gone; now on net Shared_Address_A6: PJ1.7 (Pin_7), U1.69 (PJ6(PCINT15))
- net PJ7 is gone; now on net Shared_Address_A7: PJ1.8 (Pin_8), U1.79 (PJ7)
- net PK0 is gone; now on net Shared_Address_A8: PK1.1 (Pin_1), U1.89 (PK0(ADC8/PCINT16))
- net PK1 is gone; now on net Shared_Address_A9: PK1.2 (Pin_2), U1.88 (PK1(ADC9/PCINT17))
- net PK2 is gone; now on net Shared_Address_A10: PK1.3 (Pin_3), U1.87 (PK2(ADC10/PCINT18))
- net PK3 is gone; now on net Shared_Address_A11: PK1.4 (Pin_4), U1.86 (PK3(ADC11/PCINT19))
- net PK4 is gone; now on net Shared_Address_A12: PK1.5 (Pin_5), U1.85 (PK4(ADC12/PCINT20))
- net PK5 is gone; now on net Shared_Address_A13: PK1.6 (Pin_6), U1.84 (PK5(ADC13/PCINT21))
- net PK6 is gone; now on net Shared_Address_A14: PK1.7 (Pin_7), U1.83 (PK6(ADC14/PCINT22))
- net PK7 is gone; now on net Shared_Address_A15: PK1.8 (Pin_8), U1.82 (PK7(ADC15/PCINT23))
- net PL0 is gone; now on net VGA data 0: PL1.1 (Pin_1), U1.35 (PL0(ICP4))
- net PL1 is gone; now on net VGA data 1: PL1.2 (Pin_2), U1.36 (PL1(ICP5))
- net PL2 is gone; now on net VGA data 2: PL1.3 (Pin_3), U1.37 (PL2(T5))
- net PL3 is gone; now on net VGA data 3: PL1.4 (Pin_4), U1.38 (PL3(OC5A))
- net PL4 is gone; now on net VGA data 4: PL1.5 (Pin_5), U1.39 (PL4(OC5B))
- net PL5 is gone; now on net VGA data 5: PL1.6 (Pin_6), U1.40 (PL5(OC5C))
- net PL6 is gone; now on net VGA data 6: PL1.7 (Pin_7), U1.41 (PL6)
- net PL7 is gone; now on net VGA data 7: PL1.8 (Pin_8), U1.42 (PL7)
- net Shared_Address_A16 is gone; now on net X16: M5.10 (A16)
- net +5V: now also M5.6 (CS2/CE2), R39.2
- net B16: no longer JP92.3 (B)
- net CTS: no longer R38.2
- net GND: now also R40.1; no longer LED6.1 (K), M5.30 (~{CS1}/~{CE1})
- net RTS: now also R38.2; no longer R39.2
- net SCL: now also LED6.1 (K)
- net S_ENABLE: now also M5.30 (~{CS1}/~{CE1}); no longer M5.6 (CS2/CE2)
- net X_HALT: now also R40.2
- net Mega_6309_data0 renamed Shared_data_D0
- net Mega_6309_data1 renamed Shared_data_D1
- net Mega_6309_data2 renamed Shared_data_D2
- net Mega_6309_data3 renamed Shared_data_D3
- net Mega_6309_data4 renamed Shared_data_D4
- net Mega_6309_data5 renamed Shared_data_D5
- net Mega_6309_data6 renamed Shared_data_D6
- net Mega_6309_data7 renamed Shared_data_D7
- net PD2: no longer names the net of PD1.3 (Pin_3), U1.45 ((RXD1/INT2)PD2)
- net PG4: no longer names the net of PG1.5 (Pin_5), U1.29 ((TOSC1)PG4)
- net PG5: no longer names the net of PG1.6 (Pin_6), U1.1 ((OC0B)PG5)
- no-connect marks 53 -> 50
Other:
- note added: "Free"
- note added: "Shared Memory"
- note added: "VGA Colors"
- moved on the sheet: C10, C11, C12, C13, C14, C15, C16, C2, C3, C4, C5, C6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
