File: HW/KiCad/MHF-001/MHF-001.kicad_pcb (KiCad board)
At the start: 2 copper layers, 99.9 x 99.9 mm, 186 parts, among them J1 VGA, J10 I2C, J11 + 5V -, J12 Reset, J13 +5V, J14 GND, J15 AREF, J16 XTAL2, J17 SDcard, J18 XTAL1, J19 AVCC, J2 PS/2, J20 SDcardpins, J23 VIN 12V, J24 AND_B1, J25 AND_B2, J26 AND_C1, J27 AND_C2, J28 AND_D1, J29 AND_D2, J3 RCA, J30 AND_Dx, J31 AND_Cx, J32 AND_Bx, J33 NOTF, J34 NOTE, J35 NOTEx, J36 NOTFx, J4 SysBus, J5 Micro, J6 SysBus, J7 SPI, J8 ISP, J9 Serial, M3 CY7C109D-10ZXI, M5 CY7C109D-10ZXI, Q1 BC107, U1 ATMEGA2560, U10 74HC245, U11 74HC245, U12 74HC245, U13 CH340G, U14 AMS1117-5.0, U15 AMS1117-3.3, U2 74HC14, U3 74LS08, U4 74HC165, U6 74AHC373, U7 74HC595, U8 74HC595, U9 74HC157, Y1 16 MHz, Y2 12 MHz

Commit message: Completed
Parts:
- added J100: x, Gilhad:PinHole_1x01_2.54xrectangle, F.Cu at (75.5, 93.8)
- added J101: x, Gilhad:PinHole_1x01_2.54xrectangle, F.Cu at (75.5, 96.3)
- added J102: x, Gilhad:PinHole_1x01_2.54xrectangle, F.Cu at (75.5, 98.8)
- added J103: x, Gilhad:PinHole_1x01_2.54xrectangle, F.Cu at (75.5, 101.4)
- added J104: x, Gilhad:PinHole_1x01_2.54xrectangle, F.Cu at (75.5, 103.9)
- added J105: x, Gilhad:PinHole_1x01_2.54xrectangle, F.Cu at (75.5, 106.5)
- added J106: x, Gilhad:PinHole_1x01_2.54xrectangle, F.Cu at (75.5, 109.0)
- added J107: +3V3, Gilhad:PinHole_1x01_2.54xrectangle, F.Cu at (78.6, 121.3)
- added J108: GND, Gilhad:PinHole_1x01_2.54xrectangle, F.Cu at (78.7, 123.7)
- added J109: +3V3, Gilhad:PinHole_1x01_2.54xrectangle, F.Cu at (73.0, 111.6)
- added J110: +5V, Gilhad:PinHole_1x01_2.54xrectangle, F.Cu at (62.8, 111.5)
- added J111: GND, Gilhad:PinHole_1x01_2.54xrectangle, F.Cu at (70.5, 111.6)
- added J112: GND, Gilhad:PinHole_1x01_2.54xrectangle, F.Cu at (60.3, 111.4)
- added J21: x, Gilhad:PinHole_1x01_2.54xrectangle, F.Cu at (57.7, 93.8)
- added J22: x, Gilhad:PinHole_1x01_2.54xrectangle, F.Cu at (55.2, 93.8)
- added J37: x, Gilhad:PinHole_1x01_2.54xrectangle, F.Cu at (57.7, 91.2)
- added J38: x, Gilhad:PinHole_1x01_2.54xrectangle, F.Cu at (57.7, 98.8)
- added J39: x, Gilhad:PinHole_1x01_2.54xrectangle, F.Cu at (57.7, 101.4)
- added J40: x, Gilhad:PinHole_1x01_2.54xrectangle, F.Cu at (57.7, 103.9)
- added J41: x, Gilhad:PinHole_1x01_2.54xrectangle, F.Cu at (57.7, 106.5)
- added J42: x, Gilhad:PinHole_1x01_2.54xrectangle, F.Cu at (57.7, 109.0)
- added J43: x, Gilhad:PinHole_1x01_2.54xrectangle, F.Cu at (60.3, 93.8)
- added J44: x, Gilhad:PinHole_1x01_2.54xrectangle, F.Cu at (55.2, 96.3)
- added J45: x, Gilhad:PinHole_1x01_2.54xrectangle, F.Cu at (57.7, 96.3)
- added J46: x, Gilhad:PinHole_1x01_2.54xrectangle, F.Cu at (60.3, 98.8)
- added J47: x, Gilhad:PinHole_1x01_2.54xrectangle, F.Cu at (60.3, 101.4)
- added J48: x, Gilhad:PinHole_1x01_2.54xrectangle, F.Cu at (60.3, 103.9)
- added J49: x, Gilhad:PinHole_1x01_2.54xrectangle, F.Cu at (60.3, 106.5)
- added J50: x, Gilhad:PinHole_1x01_2.54xrectangle, F.Cu at (60.3, 109.0)
- added J51: x, Gilhad:PinHole_1x01_2.54xrectangle, F.Cu at (62.8, 93.8)
- added J52: x, Gilhad:PinHole_1x01_2.54xrectangle, F.Cu at (62.8, 91.2)
- added J53: x, Gilhad:PinHole_1x01_2.54xrectangle, F.Cu at (60.3, 96.3)
- added J54: x, Gilhad:PinHole_1x01_2.54xrectangle, F.Cu at (62.8, 98.8)
- added J55: x, Gilhad:PinHole_1x01_2.54xrectangle, F.Cu at (62.8, 101.4)
- added J56: x, Gilhad:PinHole_1x01_2.54xrectangle, F.Cu at (62.8, 103.9)
- added J57: x, Gilhad:PinHole_1x01_2.54xrectangle, F.Cu at (62.8, 106.5)
- added J58: x, Gilhad:PinHole_1x01_2.54xrectangle, F.Cu at (62.8, 109.0)
- added J59: x, Gilhad:PinHole_1x01_2.54xrectangle, F.Cu at (60.3, 91.2)
- added J60: x, Gilhad:PinHole_1x01_2.54xrectangle, F.Cu at (55.2, 98.8)
- added J61: x, Gilhad:PinHole_1x01_2.54xrectangle, F.Cu at (62.8, 96.3)
- added J62: x, Gilhad:PinHole_1x01_2.54xrectangle, F.Cu at (65.4, 98.8)
- added J63: x, Gilhad:PinHole_1x01_2.54xrectangle, F.Cu at (65.4, 101.4)
- added J64: x, Gilhad:PinHole_1x01_2.54xrectangle, F.Cu at (65.4, 103.9)
- added J65: x, Gilhad:PinHole_1x01_2.54xrectangle, F.Cu at (65.4, 106.5)
- added J66: x, Gilhad:PinHole_1x01_2.54xrectangle, F.Cu at (65.4, 109.0)
- added J67: x, Gilhad:PinHole_1x01_2.54xrectangle, F.Cu at (65.4, 91.2)
- added J68: x, Gilhad:PinHole_1x01_2.54xrectangle, F.Cu at (65.4, 93.8)
- added J69: x, Gilhad:PinHole_1x01_2.54xrectangle, F.Cu at (65.4, 96.3)
- added J70: x, Gilhad:PinHole_1x01_2.54xrectangle, F.Cu at (67.9, 98.8)
- added J71: x, Gilhad:PinHole_1x01_2.54xrectangle, F.Cu at (67.9, 101.4)
- added J72: x, Gilhad:PinHole_1x01_2.54xrectangle, F.Cu at (67.9, 103.9)
- added J73: x, Gilhad:PinHole_1x01_2.54xrectangle, F.Cu at (67.9, 106.5)
- added J74: x, Gilhad:PinHole_1x01_2.54xrectangle, F.Cu at (67.9, 109.0)
- added J75: x, Gilhad:PinHole_1x01_2.54xrectangle, F.Cu at (67.9, 91.2)
- added J76: x, Gilhad:PinHole_1x01_2.54xrectangle, F.Cu at (67.9, 93.8)
- added J77: x, Gilhad:PinHole_1x01_2.54xrectangle, F.Cu at (67.9, 96.3)
- added J78: x, Gilhad:PinHole_1x01_2.54xrectangle, F.Cu at (70.4, 98.8)
- added J79: x, Gilhad:PinHole_1x01_2.54xrectangle, F.Cu at (70.4, 101.4)
- added J80: x, Gilhad:PinHole_1x01_2.54xrectangle, F.Cu at (70.4, 103.9)
- added J81: x, Gilhad:PinHole_1x01_2.54xrectangle, F.Cu at (70.4, 106.5)
- added J82: x, Gilhad:PinHole_1x01_2.54xrectangle, F.Cu at (70.4, 109.0)
- added J83: x, Gilhad:PinHole_1x01_2.54xrectangle, F.Cu at (55.2, 104.0)
- added J84: x, Gilhad:PinHole_1x01_2.54xrectangle, F.Cu at (70.4, 93.8)
- added J85: x, Gilhad:PinHole_1x01_2.54xrectangle, F.Cu at (70.4, 96.3)
- added J86: x, Gilhad:PinHole_1x01_2.54xrectangle, F.Cu at (55.2, 101.4)
- added J87: x, Gilhad:PinHole_1x01_2.54xrectangle, F.Cu at (75.4, 91.3)
- added J88: x, Gilhad:PinHole_1x01_2.54xrectangle, F.Cu at (55.2, 106.5)
- added J89: x, Gilhad:PinHole_1x01_2.54xrectangle, F.Cu at (55.2, 91.2)
- added J90: x, Gilhad:PinHole_1x01_2.54xrectangle, F.Cu at (55.3, 109.0)
- added J91: x, Gilhad:PinHole_1x01_2.54xrectangle, F.Cu at (73.0, 93.8)
- added J92: x, Gilhad:PinHole_1x01_2.54xrectangle, F.Cu at (70.4, 91.2)
- added J93: x, Gilhad:PinHole_1x01_2.54xrectangle, F.Cu at (73.0, 96.3)
- added J94: x, Gilhad:PinHole_1x01_2.54xrectangle, F.Cu at (73.0, 98.8)
- added J95: x, Gilhad:PinHole_1x01_2.54xrectangle, F.Cu at (73.0, 101.4)
- added J96: x, Gilhad:PinHole_1x01_2.54xrectangle, F.Cu at (73.0, 103.9)
- added J97: x, Gilhad:PinHole_1x01_2.54xrectangle, F.Cu at (73.0, 106.5)
- added J98: x, Gilhad:PinHole_1x01_2.54xrectangle, F.Cu at (73.0, 109.0)
- added J99: x, Gilhad:PinHole_1x01_2.54xrectangle, F.Cu at (73.0, 91.2)
- U14: value AMS1117-5.0 -> 5.0V
- U15: value AMS1117-3.3 -> 3.3 V
Routing:
- net GND: track 847.1 -> 893.0 mm
- net +5V: track 740.4 -> 782.4 mm, vias 11 -> 15
- net S_ENABLE: track 76.9 -> 45.4 mm, vias 0 -> 2
- net VGA data 2: track 76.6 -> 55.5 mm, vias 1 -> 2
- net S_READ: track 65.9 -> 47.8 mm, vias 0 -> 2
- net +3.3V: track 12.1 -> 27.6 mm
- net RTS: track 68.0 -> 55.8 mm, vias 1 -> 3
- net Reset: track 125.3 -> 116.0 mm, vias 3 -> 5
- net SIGNAL_RCA: track 116.9 -> 125.7 mm
- net HSyncVGA: track 147.4 -> 152.9 mm
- net XAA5: track 69.4 -> 64.1 mm, vias 1 -> 3
- net Net-(PG1-Pin_5): track 41.4 -> 36.5 mm, vias 1 -> 3
- net RX: track 56.9 -> 52.4 mm, vias 1 -> 2
- net MISO: track 84.8 -> 89.2 mm
- net VGA Latch: track 139.4 -> 143.0 mm
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