File: HW/KiCad/MHF-002/MHF-002.kicad_sch (KiCad schematic)
At the start: 289 parts, among them J1 VGA, J10 I2C, J100 x, J101 x, J102 x, J103 x, J104 x, J105 x, J106 x, J107 +3V3, J108 GND, J109 +3V3, J11 + 5V -, J110 +5V, J111 GND, J112 GND, J113 SDCard, J12 Reset, J13 +5V, J14 GND, J15 AREF, J16 XTAL2, J17 SDcard, J18 XTAL1, J19 AVCC, J2 PS/2, J20 SDcardpins, J21 x, J22 x, J23 VIN 12V, J24 AND_B1, J25 AND_B2, J26 AND_C1, J27 AND_C2, J28 AND_D1, J29 AND_D2, J3 RCA, J30 AND_Dx, J31 AND_Cx, J32 AND_Bx, J33 NOTF, J34 NOTE, J35 NOTEx, J36 NOTFx, J37 x, J38 x, J39 x, J4 SysBus, J40 x, J41 x, J42 x, J43 x, J44 x, J45 x, J46 x, J47 x, J48 x, J49 x, J5 Micro, J50 x, J51 x, J52 x, J53 x, J54 x, J55 x, J56 x, J57 x, J58 x, J59 x, J6 SysBus, J60 x, J61 x, J62 x, J63 x, J64 x, J65 x, J66 x, J67 x, J68 x, J69 x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

Commit message: footprints (maybe complete)
Parts:
- C1: footprint Capacitor_THT:C_Disc_D4.3mm_W1.9mm_P5.00mm -> MHF:C_Disc_D4.3mm_W1.9mm_P5.00mm
- C10, C11, C13, C14, C15, C16, C2, C5, C6, C7, C8: footprint Capacitor_SMD:C_0603_1608Metric_Pad1.08x0.95mm_HandSolder -> MHF:C_0805_2012Metric_HandSolder
- C12, C9, Cx1, Cx10, Cx11, Cx12, Cx13, Cx2, Cx3, Cx4, Cx5, Cx6, Cx7, Cx8, Cx9: footprint Capacitor_THT:C_Disc_D3.0mm_W2.0mm_P2.50mm -> MHF:C_Disc_D3.0mm_W2.0mm_P2.50mm
- C3, C4: value 100n -> 22n; footprint Capacitor_SMD:C_0603_1608Metric_Pad1.08x0.95mm_HandSolder -> MHF:C_0805_2012Metric_HandSolder
- Cx14, Cx15: footprint Capacitor_THT:CP_Radial_D5.0mm_P2.50mm -> MHF:CP_Radial_D5.0mm_P2.50mm
- D1: footprint Diode_THT:D_DO-41_SOD81_P10.16mm_Horizontal -> MHF:D_DO-41_SOD81_P10.16mm_Horizontal
- D2: footprint Diode_SMD:D_1206_3216Metric -> MHF:D_1210_3225Metric_HandSolder
- D3: footprint Diode_SMD:D_1210_3225Metric -> MHF:D_1210_3225Metric_HandSolder
- F1: footprint Fuse:Fuse_1206_3216Metric_Pad1.42x1.75mm_HandSolder -> MHF:Fuse_1206_3216Metric_Pad1.42x1.75mm_HandSolder
- H5, H6, H7, H8: footprint MountingHole:MountingHole_3.2mm_M3_Pad -> MHF:MountingHole_3.2mm_M3_Pad
- J1: footprint Connector_Dsub:DSUB-15-HD_Socket_Horizontal_P2.29x2.54mm_EdgePinOffset8.35mm_Housed_MountingHolesOffset10.89mm -> MHF:DSUB-15-HD_Socket_Horizontal_P2.29x2.54mm_EdgePinOffset8.35mm_Housed_MountingHolesOffset10.89mm
- J10, J20: footprint Connector_PinHeader_2.54mm:PinHeader_1x04_P2.54mm_Vertical -> MHF:PinHeader_1x04_P2.54mm_Vertical
- J100, J101, J102, J103, J104, J105, J106, J107, J108, J109, J110, J111, J112, J12, J13, J14, J15, J16, J18, J19, J21, J22, J24, J25, J26, J27, J28, J29, J30, J31, J32, J33, J34, J35, J36, J37, J38, J39, J40, J41, J42, J43, J44, J45, J46, J47, J48, J49, J50, J51, J52, J53, J54, J55, J56, J57, J58, J59, J60, J61, J62, J63, J64, J65, J66, J67, J68, J69, J70, J71, J72, J73, J74, J75, J76, J77, J78, J79, J80, J81, J82, J83, J84, J85, J86, J87, J88, J89, J90, J91, J92, J93, J94, J95, J96, J97, J98, J99: footprint Gilhad:PinHole_1x01_2.54xrectangle -> MHF:PinHole_1x01_2.54xrectangle
- J11: footprint Connector_PinSocket_2.54mm:PinSocket_2x03_P2.54mm_Vertical -> MHF:PinSocket_2x03_P2.54mm_Vertical
- J17, J7, J9, JP27, PG1: footprint Connector_PinHeader_2.54mm:PinHeader_1x06_P2.54mm_Vertical -> MHF:PinHeader_1x06_P2.54mm_Vertical
- J23: footprint Connector_BarrelJack:BarrelJack_Horizontal -> MHF:BarrelJack_Horizontal
- J4: footprint Connector_PinSocket_2.54mm:PinSocket_2x32_P2.54mm_Vertical -> MHF:PinSocket_2x32_P2.54mm_Vertical
- J5: footprint Connector_USB:USB_Micro-B_XKB_U254-051T-4BH83-F1S -> MHF:USB_Micro-B_XKB_U254-051T-4BH83-F1S
- J6: footprint Connector_PinHeader_2.54mm:PinHeader_2x32_P2.54mm_Vertical -> MHF:PinHeader_2x32_P2.54mm_Vertical
- J8: footprint Connector_PinHeader_2.54mm:PinHeader_2x03_P2.54mm_Vertical -> MHF:PinHeader_2x03_P2.54mm_Vertical
- JP1, JP10, JP11, JP12, JP13, JP14, JP2, JP3, JP4, JP5, JP6, JP7, JP8, JP9, JP91: footprint Jumper:SolderJumper-2_P1.3mm_Bridged_Pad1.0x1.5mm -> MHF:SolderJumper-2_P1.3mm_Bridged_Pad1.0x1.5mm
- JP100, JP102, JP103, JP104, JP105, JP106, JP107, JP92, JP94, JP95, JP98, JP99: footprint Jumper:SolderJumper-3_P1.3mm_Open_RoundedPad1.0x1.5mm -> MHF:SolderJumper-3_P1.3mm_Open_RoundedPad1.0x1.5mm
- JP15, JP16, JP17, JP18, JP19, JP21, JP22, JP23, JP24, JP25, JP55, JP56: footprint Jumper:SolderJumper-2_P1.3mm_Open_RoundedPad1.0x1.5mm -> MHF:SolderJumper-2_P1.3mm_Open_RoundedPad1.0x1.5mm
- JP26, JP28: footprint Connector_PinHeader_2.54mm:PinHeader_1x02_P2.54mm_Vertical -> MHF:PinHeader_1x02_P2.54mm_Vertical
- LED1, LED10, LED2, LED3, LED4, LED5, LED6, LED7, LED8, LED9: footprint LED_SMD:LED_0805_2012Metric -> MHF:LED_0805_2012Metric
- N1, N3: footprint NetTie:NetTie-2_SMD_Pad0.5mm -> MHF:NetTie-2_SMD_Pad0.5mm
- PA1, PB1, PC1, PD1, PE1, PF1, PH1, PJ1, PK1, PL1: footprint Connector_PinHeader_2.54mm:PinHeader_1x08_P2.54mm_Vertical -> MHF:PinHeader_1x08_P2.54mm_Vertical
- Q1: footprint Package_TO_SOT_THT:TO-92_Inline -> MHF:TO-92_Inline
- R1, R10, R11, R12, R13, R14, R15, R16, R17, R18, R19, R2, R20, R21, R22, R23, R3, R32, R33, R38, R39, R4, R41, R43, R44, R45, R46, R47, R5, R6, R7, R8, R9: footprint Resistor_SMD:R_0805_2012Metric_Pad1.20x1.40mm_HandSolder -> MHF:R_0805_2012Metric_Pad1.20x1.40mm_HandSolder
- R24, R25, R26, R27, R28, R29, R30, R31, R34, R35, R36, R37, R40: footprint Resistor_SMD:R_0603_1608Metric_Pad0.98x0.95mm_HandSolder -> MHF:R_0805_2012Metric_Pad1.20x1.40mm_HandSolder
- R42: footprint Resistor_SMD:R_0603_1608Metric_Pad0.98x0.95mm_HandSolder -> MHF:R_0805_2012Metric_Pad1.20x1.40mm_HandSolder; now fitted
- U13: footprint Package_SO:SOIC-16_3.9x9.9mm_P1.27mm -> MHF:SOIC-16_3.9x9.9mm_P1.27mm
- U14, U15: footprint Package_TO_SOT_SMD:SOT-223-3_TabPin2 -> MHF:SOT-223-3_TabPin2_HandSolder
- U2, U3: footprint Package_DIP:DIP-14_W7.62mm -> MHF:SOIC-14_3.9x8.7mm_P1.27mm
- U4: footprint Package_SO:TSSOP-20_4.4x5mm_P0.5mm -> MHF:TSSOP-20_4.4x6.5mm_P0.65mm_HandSolder
- U5: footprint MHF:G_SOIC-16_3.9x9.9mm_HandSolder -> MHF:SOIC-16_3.9x9.9mm_P1.27mm
- U7, U8, U9: footprint Package_DIP:DIP-16_W7.62mm -> MHF:SOIC-16_3.9x9.9mm_P1.27mm
- Y1, Y2: footprint Crystal:Crystal_SMD_HC49-SD -> MHF:Crystal_SMD_HC49-SD
Connections:
- net GND: now also J2.S (Shield)
- net L0: now also M3.20 (A0), U4.19 (Q0); no longer M3.17 (A3), U4.16 (Q3)
- net L1: now also M3.19 (A1), U4.18 (Q1); no longer M3.18 (A2), U4.17 (Q2)
- net L2: now also M3.18 (A2), U4.17 (Q2); no longer M3.19 (A1), U4.18 (Q1)
- net L3: now also M3.17 (A3), U4.16 (Q3); no longer M3.20 (A0), U4.19 (Q0)
- net L4: now also M3.13 (A7); no longer M3.16 (A4)
- net L5: now also M3.14 (A6); no longer M3.15 (A5)
- net L6: now also M3.15 (A5); no longer M3.14 (A6)
- net L7: now also M3.16 (A4); no longer M3.13 (A7)
- net XAD0: now also U4.9 (D7); no longer U4.5 (D3)
- net XAD1: now also U4.8 (D6); no longer U4.4 (D2)
- net XAD2: now also U4.7 (D5); no longer U4.3 (D1)
- net XAD3: now also U4.6 (D4); no longer U4.2 (D0)
- net XAD4: now also U4.5 (D3); no longer U4.6 (D4)
- net XAD5: now also U4.4 (D2); no longer U4.7 (D5)
- net XAD6: now also U4.3 (D1); no longer U4.8 (D6)
- net XAD7: now also U4.2 (D0); no longer U4.9 (D7)
Other:
- moved on the sheet: M3, U4
