File: HW/KiCad/MHF-002/MHF-002.kicad_sch (KiCad schematic)
At the start: 289 parts, among them J1 VGA, J10 I2C, J100 x, J101 x, J102 x, J103 x, J104 x, J105 x, J106 x, J107 +3V3, J108 GND, J109 +3V3, J11 + 5V -, J110 +5V, J111 GND, J112 GND, J113 SDCard, J12 Reset, J13 +5V, J14 GND, J15 AREF, J16 XTAL2, J17 SDcard, J18 XTAL1, J19 AVCC, J2 PS/2, J20 SDcardpins, J21 x, J22 x, J23 VIN 12V, J24 AND_B1, J25 AND_B2, J26 AND_C1, J27 AND_C2, J28 AND_D1, J29 AND_D2, J3 RCA, J30 AND_Dx, J31 AND_Cx, J32 AND_Bx, J33 NOTF, J34 NOTE, J35 NOTEx, J36 NOTFx, J37 x, J38 x, J39 x, J4 SysBus, J40 x, J41 x, J42 x, J43 x, J44 x, J45 x, J46 x, J47 x, J48 x, J49 x, J5 Micro, J50 x, J51 x, J52 x, J53 x, J54 x, J55 x, J56 x, J57 x, J58 x, J59 x, J6 SysBus, J60 x, J61 x, J62 x, J63 x, J64 x, J65 x, J66 x, J67 x, J68 x, J69 x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

Commit message: included all planned improvements
Parts:
- added D10, D11, D4, D5, D6, D7, D8, D9: WS2812B, MHF:LED_WS2812B_PLCC4_5.0x5.0mm_P3.2mm_HandSolder, symbol MHF:WS2812B
- added J114: VIN, MHF:PinHole_1x01_2.54xrectangle, symbol MHF:Conn_01x01
- added J115: VI, MHF:PinHole_1x01_2.54xrectangle, symbol MHF:Conn_01x01
- added J116: GND, MHF:PinHole_1x01_2.54xrectangle, symbol MHF:Conn_01x01
- added JP29: SBC_D_Dir, MHF:SolderJumper-2_P1.3mm_Open_RoundedPad1.0x1.5mm, symbol MHF:SolderJumper_2_Open
- added JP33: SBC_A_DIR, MHF:SolderJumper-2_P1.3mm_Open_RoundedPad1.0x1.5mm, symbol MHF:SolderJumper_2_Open
- added JP34: SBC_G_Enable, MHF:SolderJumper-2_P1.3mm_Open_RoundedPad1.0x1.5mm, symbol MHF:SolderJumper_2_Open
- added JP35: SBC_S_Enable, MHF:SolderJumper-2_P1.3mm_Open_RoundedPad1.0x1.5mm, symbol MHF:SolderJumper_2_Open
- added JP36: SBC_Read, MHF:SolderJumper-2_P1.3mm_Open_RoundedPad1.0x1.5mm, symbol MHF:SolderJumper_2_Open
- added JP37: SBC_Write, MHF:SolderJumper-2_P1.3mm_Open_RoundedPad1.0x1.5mm, symbol MHF:SolderJumper_2_Open
- added R48, R49: 1k, MHF:R_0805_2012Metric_Pad1.20x1.40mm_HandSolder, symbol MHF:R
- J9, PG1: footprint MHF:PinHeader_1x06_P2.54mm_Vertical -> MHF:PinHeader_1x07_P2.54mm_Vertical; symbol MHF:Conn_01x06 -> MHF:Conn_01x07
- JP92: value X16 -> X_S16
- PA1, PB1, PC1, PD1, PE1, PF1, PH1, PJ1, PK1, PL1: footprint MHF:PinHeader_1x08_P2.54mm_Vertical -> MHF:PinHeader_1x09_P2.54mm_Vertical; symbol MHF:Conn_01x08 -> MHF:Conn_01x09
Connections:
- net +5V: now also J9.7 (Pin_7), D10.1 (VDD), D11.1 (VDD), D4.1 (VDD), D5.1 (VDD), D6.1 (VDD), D7.1 (VDD), D8.1 (VDD), D9.1 (VDD); no longer J9.6 (Pin_6)
- net DTR: now also J9.5 (Pin_5)
- net GND: now also J9.6 (Pin_6), PA1.9 (Pin_9), PB1.9 (Pin_9), PC1.9 (Pin_9), PD1.9 (Pin_9), PE1.9 (Pin_9), PF1.9 (Pin_9), PG1.7 (Pin_7), PH1.9 (Pin_9), PJ1.9 (Pin_9), PK1.9 (Pin_9), PL1.9 (Pin_9), D10.3 (VSS), D11.3 (VSS), D4.3 (VSS), D5.3 (VSS), D6.3 (VSS), D7.3 (VSS), D8.3 (VSS), D9.3 (VSS), J116.1 (Pin_1); no longer J9.5 (Pin_5)
- net G_A_DIR: now also JP33.2 (B)
- net G_D_DIR: now also JP29.2 (B)
- net G_ENABLE: now also JP34.2 (B)
- net MISO: now also JP55.1 (A)
- net SCK: no longer JP55.1 (A)
- net S_ENABLE: now also JP35.2 (B)
- net S_READ: now also JP36.2 (B)
- net S_WRITE: now also JP37.2 (B)
- net VIN: now also J114.1 (Pin_1)
- net X_HALT: now also JP37.1 (A)
- net X_READ: now also JP36.1 (A)
- net X_SHARE_DIRTY: now also JP35.1 (A)
- net X_SHARE_GRANTED: now also JP29.1 (A), R48.2; no longer PD1.5 (Pin_5), U1.47 ((ICP1)PD4)
- net X_SHARE_REQUEST: now also PG1.5 (Pin_5), U1.29 ((TOSC1)PG4), JP33.1 (A); no longer PD1.6 (Pin_6), U1.48 ((XCK1)PD5)
- net X_SHARE_FUTURE: now reaches PG1.6 (Pin_6), U1.1 ((OC0B)PG5)
- net X_SHARE_FUTURE: now also JP34.1 (A)
- net at C11.1, D3.1 (K), U14.3 (VI): now also J115.1 (Pin_1)
- net X16 renamed X_S16
- new net: D8.2 (DOUT), D9.4 (DIN)
- new net: D7.2 (DOUT), D8.4 (DIN)
- new net: D10.2 (DOUT), D11.4 (DIN)
- new net: D10.4 (DIN), D9.2 (DOUT)
- new net: PD1.5 (Pin_5), R48.1, R49.1, U1.47 ((ICP1)PD4)
- new net: PD1.6 (Pin_6), U1.48 ((XCK1)PD5)
- new net: D6.2 (DOUT), D7.4 (DIN)
- new net: D4.2 (DOUT), D5.4 (DIN)
- new net: D5.2 (DOUT), D6.4 (DIN)
- new net Debug_LEDs: D4.4 (DIN), R49.2
- no-connect marks 126 -> 127
Other:
- note added: "SCK for Sigral_RCA"
- note removed: "Free"
- moved on the sheet: C12, C9, D2, J113, J12, J17, J20, J23, JP1, JP2, JP3, JP4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

Commit message: MHF-002 routing full PCB, need add texts
Parts:
- removed J20: SDcardpins, MHF:PinHeader_1x04_P2.54mm_Vertical, symbol MHF:Conn_01x04
- C12: value 100n -> 100n RESET
- C9: value 100n -> 100n DTR
- D1: footprint MHF:D_DO-41_SOD81_P10.16mm_Horizontal -> MHF:D_DO-41_SOD81_P9.4mm_Horizontal
- LED1: value RX -> RX0
- LED2: value TX -> TX0
- LED4: value CTS -> CTS0
- LED5: value RTS -> RTS0
- R37, R46: value 10k -> 1k
Connections:
- net DTR: now also J9.3 (Pin_3); no longer J9.5 (Pin_5)
- net at JP15.1 (A): now also R30.1; no longer U13.2 (TXD)
- net at JP16.1 (A): now also R31.1; no longer U13.3 (RXD)
- net CTS renamed CTS0
- net CTS0: now also JP19.2 (B), JP25.2 (B); no longer JP17.2 (B), JP23.2 (B)
- net M8RXD renamed TX0
- net TX0: now also J9.5 (Pin_5), LED2.1 (K), PE1.2 (Pin_2), U1.3 ((TXD0)PE1); no longer LED1.1 (K), R30.2
- net M8TXD renamed RX0
- net RX0: now also J9.4 (Pin_4), LED1.1 (K), PE1.1 (Pin_1), U1.2 ((RXD0/PCIN8)PE0); no longer LED2.1 (K), R31.2
- net RTS renamed RTS0
- net RTS0: now also JP17.2 (B), JP23.2 (B); no longer JP19.2 (B), JP25.2 (B)
- removed net RX: J9.3 (Pin_3), PE1.2 (Pin_2), R30.1, U1.3 ((TXD0)PE1)
- removed net TX: J9.4 (Pin_4), PE1.1 (Pin_1), R31.1, U1.2 ((RXD0/PCIN8)PE0)
- new net: R31.2, U13.3 (RXD)
- new net: R30.2, U13.2 (TXD)

Commit message: improved SystemBus and 3xAND, NOT
Parts:
- removed D10, D11: WS2812B, MHF:LED_WS2812B_PLCC4_5.0x5.0mm_P3.2mm_HandSolder, symbol MHF:WS2812B
- C9: value 100n DTR -> DTR 100n
- J6: footprint MHF:PinHeader_2x32_P2.54mm_Vertical -> MHF:PinHeader_2x32_P2.54mm_Vertical_down
- JP13: value Xhalt -> XHalt
- PA1: value PA0 -> PA
- PB1: value PB0 -> PB
- PC1: value PC0 -> PC
- PD1: value PD0 -> PD
- PE1: value PE0 -> PE
- PF1: value PF0 -> PF
- PG1: value PG0 -> PG
- PH1: value PH0 -> PH
- PJ1: value PJ0 -> PJ
- PK1: value PK0 -> PK
- PL1: value PL0 -> PL
- R40: value 1k -> HALTdown 1k
- R42: value 1k -> HALTup 1k

Commit message: D-Latch testpoints
Parts:
- added TP1: 7, MHF:TestPoint_Pad_1.0x1.0mm, symbol MHF:TestPoint_Probe
- added TP2: 0, MHF:TestPoint_Pad_1.0x1.0mm, symbol MHF:TestPoint_Probe
- added TP3: 1, MHF:TestPoint_Pad_1.0x1.0mm, symbol MHF:TestPoint_Probe
- added TP4: 2, MHF:TestPoint_Pad_1.0x1.0mm, symbol MHF:TestPoint_Probe
- added TP5: 3, MHF:TestPoint_Pad_1.0x1.0mm, symbol MHF:TestPoint_Probe
- added TP6: 4, MHF:TestPoint_Pad_1.0x1.0mm, symbol MHF:TestPoint_Probe
- added TP7: 5, MHF:TestPoint_Pad_1.0x1.0mm, symbol MHF:TestPoint_Probe
- added TP8: 6, MHF:TestPoint_Pad_1.0x1.0mm, symbol MHF:TestPoint_Probe
- C1: value 10 nF -> 10nF
Connections:
- net A_G_D_DIR: now also J4.49 (Pin_49), J6.49 (Pin_49); no longer J4.45 (Pin_45), J6.45 (Pin_45)
- net A_G_ENABLE: now also J4.45 (Pin_45), J6.45 (Pin_45); no longer J4.49 (Pin_49), J6.49 (Pin_49)
- net B_G_D_DIR: now also J4.50 (Pin_50), J6.50 (Pin_50); no longer J4.46 (Pin_46), J6.46 (Pin_46)
- net B_G_ENABLE: now also J4.46 (Pin_46), J6.46 (Pin_46); no longer J4.50 (Pin_50), J6.50 (Pin_50)
- net GND: now also J1.0
- net L0: now also TP1.1
- net L1: now also TP8.1
- net L2: now also TP7.1
- net L3: now also TP6.1
- net L4: now also TP5.1
- net L5: now also TP4.1
- net L6: now also TP3.1
- net L7: now also TP2.1
- no-connect marks 127 -> 126

Commit message: reset + I2C LED
Parts:
- added Cx16, Cx17, Cx18: Cx, MHF:C_Disc_D3.0mm_W2.0mm_P2.50mm, symbol MHF:C
- added D10: SS14, MHF:D_1812_4532Metric_Pad1.30x3.40mm_HandSolder, symbol MHF:D
- added Q2: 2907, MHF:TSOT-23_HandSoldering, symbol MHF:PNP
- JP26: value PS/2 -> PS2
- R40: value HALTdown 1k -> 1k
- R42: value HALTup 1k -> 1k
Connections:
- net +5V: now also Cx16.1, Cx17.1, Cx18.1
- net GND: now also Cx16.2, Cx17.2, Cx18.2, Q2.3 (C)
- net L0: now also M3.16 (A4), TP2.1, U4.12 (Q7); no longer M3.20 (A0), TP1.1, U4.19 (Q0)
- net L1: now also M3.15 (A5), TP3.1, U4.13 (Q6); no longer M3.19 (A1), TP8.1, U4.18 (Q1)
- net L2: now also M3.14 (A6), TP4.1, U4.14 (Q5); no longer M3.18 (A2), TP7.1, U4.17 (Q2)
- net L3: now also M3.13 (A7), TP5.1, U4.15 (Q4); no longer M3.17 (A3), TP6.1, U4.16 (Q3)
- net L4: now also M3.17 (A3), TP6.1, U4.16 (Q3); no longer M3.13 (A7), TP5.1, U4.15 (Q4)
- net L5: now also M3.18 (A2), TP7.1, U4.17 (Q2); no longer M3.14 (A6), TP4.1, U4.14 (Q5)
- net L6: now also M3.19 (A1), TP8.1, U4.18 (Q1); no longer M3.15 (A5), TP3.1, U4.13 (Q6)
- net L7: now also M3.20 (A0), TP1.1, U4.19 (Q0); no longer M3.16 (A4), TP2.1, U4.12 (Q7)
- net Reset: now also D10.2 (A)
- net SCL: now also Q2.1 (B); no longer LED6.1 (K)
- net MasterReset: now reaches J6.62 (Pin_62)
- net MasterReset: now also J4.62 (Pin_62), D10.1 (K)
- new net: LED6.1 (K), Q2.2 (E)
- no-connect marks 126 -> 124
Other:
- moved on the sheet: D2, J12, R26

Commit message: Final version of HW MHF-002
Parts:
- JP14: value AVCC -> xAVCC
- JP21: value TX2102 -> RX0
- JP22: value RX2102 -> TX0
- JP23: value CTS2102 -> RTS0
- JP24: value DTR2102 -> DTR0
- JP25: value RTS2102 -> CTS0
Other:
- moved on the sheet: U2F

Commit message: redesigned PS/2 and RCA to 40/80 char sources, need route
Parts:
- added J20: RCAsel, MHF:PinHeader_1x03_P2.54mm_Vertical, symbol MHF:Conn_01x03
Connections:
- net Bb: no longer R17.2
- net Bf: no longer R21.2
- net GND: no longer U9.15 (E)
- net Gb: no longer R18.2
- net Gf: no longer R22.2
- net HSyncVGA: now also N3.2
- net Ib: no longer R16.2
- net If: no longer R20.2
- net Rb: no longer R19.2
- net Rf: no longer R23.2
- net SIGNAL_RCA: now also J20.1 (Pin_1); no longer R5.1, U3.1
- net VGA data 0: now also R16.2
- net VGA data 1: now also R17.2
- net VGA data 2: now also R18.2
- net VGA data 3: now also R19.2; no longer N3.2
- net VGA data 4: now also R20.2
- net VGA data 5: now also R21.2
- net VGA data 6: now also R22.2
- net VGA data 7: now also R23.2
- net ~{VGA_Enable}: now reaches PD1.3 (Pin_3), U1.45 ((RXD1/INT2)PD2)
- net ~{VGA_Enable}: now also U9.15 (E)
- net at U5.13 (Qh), U9.1 (S): now also J20.3 (Pin_3)
- new net: J20.2 (Pin_2), R5.1, U3.1
Other:
- note added: "SCK for Signal_RCA"
- note removed: "SCK for Sigral_RCA"

Commit message: renumbered RAMs
Connections:
- net Shared_data_D0: now also M5.29 (DQ7); no longer M5.21 (DQ0)
- net Shared_data_D1: now also M5.28 (DQ6); no longer M5.22 (DQ1)
- net Shared_data_D2: now also M5.27 (DQ5); no longer M5.23 (DQ2)
- net Shared_data_D3: now also M5.26 (DQ4); no longer M5.25 (DQ3)
- net Shared_data_D4: now also M5.25 (DQ3); no longer M5.26 (DQ4)
- net Shared_data_D5: now also M5.23 (DQ2); no longer M5.27 (DQ5)
- net Shared_data_D6: now also M5.22 (DQ1); no longer M5.28 (DQ6)
- net Shared_data_D7: now also M5.21 (DQ0); no longer M5.29 (DQ7)
- net XAA0: now also M3.1 (A11); no longer M3.3 (A8)
- net XAA2: now also M3.3 (A8); no longer M3.31 (A10)
- net XAA3: now also M3.4 (A13); no longer M3.1 (A11)
- net XAA4: now also M3.7 (A15); no longer M3.12 (A12)
- net XAA5: now also M3.11 (A14); no longer M3.4 (A13)
- net XAA6: now also M3.12 (A12); no longer M3.11 (A14)
- net XAA7: now also M3.31 (A10); no longer M3.7 (A15)
Changed lines of the file:
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@@
 		)
 	)
-	(label "XAA4"
+	(label "XAA6"
 		(at 675.64 386.08 180)
 		(effects
@@
 		)
 	)
-	(label "Shared_data_D6"
+	(label "Shared_data_D1"
 		(at 250.19 429.26 180)
 		(effects
@@
 		)
 	)
-	(label "Shared_data_D5"
+	(label "Shared_data_D2"
 		(at 250.19 426.72 180)
 		(effects
@@
 		)
 	)
-	(label "Shared_data_D2"
+	(label "Shared_data_D5"
 		(at 250.19 419.1 180)
 		(effects
@@
 		)
 	)
-	(label "Shared_data_D4"
+	(label "Shared_data_D3"
 		(at 250.19 424.18 180)
 		(effects
@@
 		)
 	)
-	(label "XAA5"
+	(label "XAA3"
 		(at 675.64 388.62 180)
 		(effects
@@
 		)
 	)
-	(label "Shared_data_D3"
+	(label "Shared_data_D4"
 		(at 250.19 421.64 180)
 		(effects
@@
 		)
 	)
-	(label "XAA0"
+	(label "XAA2"
 		(at 675.64 375.92 180)
 		(effects
@@
 		)
 	)
-	(label "XAA2"
+	(label "XAA7"
 		(at 675.64 381 180)
 		(effects
@@
 		)
 	)
-	(label "Shared_data_D1"
+	(label "Shared_data_D6"
 		(at 250.19 416.56 180)
 		(effects
@@
 		)
 	)
-	(label "Shared_data_D0"
+	(label "Shared_data_D7"
 		(at 250.19 414.02 180)
 		(effects
@@
 		)
 	)
-	(label "Shared_data_D7"
+	(label "Shared_data_D0"
 		(at 250.19 431.8 180)
 		(effects
@@
 		)
 	)
-	(label "XAA3"
+	(label "XAA0"
 		(at 675.64 383.54 180)
 		(effects
@@
 		)
 	)
-	(label "XAA7"
+	(label "XAA4"
 		(at 675.64 393.7 180)
 		(effects
@@
 		)
 	)
-	(label "XAA6"
+	(label "XAA5"
 		(at 675.64 391.16 180)
 		(effects
