File: HW/KiCad/MHF-002/MHF-002.kicad_sch (KiCad schematic)
At the start: 319 parts, among them J1 VGA, J10 I2C, J100 x, J101 x, J102 x, J103 x, J104 x, J105 x, J106 x, J107 +3V3, J108 GND, J109 +3V3, J11 + 5V -, J110 +5V, J111 GND, J112 GND, J113 SDCard, J114 VIN, J115 VI, J116 GND, J12 Reset, J13 +5V, J14 GND, J15 AREF, J16 XTAL2, J17 SDcard, J18 XTAL1, J19 AVCC, J2 PS/2, J20 RCAsel, J21 x, J22 x, J23 VIN 12V, J24 AND_B1, J25 AND_B2, J26 AND_C1, J27 AND_C2, J28 AND_D1, J29 AND_D2, J3 RCA, J30 AND_Dx, J31 AND_Cx, J32 AND_Bx, J33 NOTF, J34 NOTE, J35 NOTEx, J36 NOTFx, J37 x, J38 x, J39 x, J4 SysBus, J40 x, J41 x, J42 x, J43 x, J44 x, J45 x, J46 x, J47 x, J48 x, J49 x, J5 Micro, J50 x, J51 x, J52 x, J53 x, J54 x, J55 x, J56 x, J57 x, J58 x, J59 x, J6 SysBus, J60 x, J61 x, J62 x, J63 x, J64 x, J65 x, J66 x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

Commit message: more renumbering
Parts:
- removed N1, N3: ~, MHF:NetTie-2_SMD_Pad0.5mm, symbol MHF:NetTie_2
Connections:
- net VSyncVGA is gone; now on net VSyncVGA_RCA: PE1.5 (Pin_5), R15.2, U1.6 ((OC3B/INT4)PE4)
- net ~{SUPRESS} is gone; now on net HSyncVGA_SuppressRCA: U3.2
- net Shared_Address_A10: now also M5.3 (A8); no longer M5.31 (A10)
- net Shared_Address_A11: now also M5.4 (A13); no longer M5.1 (A11)
- net Shared_Address_A12: now also M5.7 (A15); no longer M5.12 (A12)
- net Shared_Address_A13: now also M5.11 (A14); no longer M5.4 (A13)
- net Shared_Address_A14: now also M5.12 (A12); no longer M5.11 (A14)
- net Shared_Address_A15: now also M5.31 (A10); no longer M5.7 (A15)
- net Shared_Address_A4: now also M5.13 (A7); no longer M5.16 (A4)
- net Shared_Address_A5: now also M5.14 (A6); no longer M5.15 (A5)
- net Shared_Address_A6: now also M5.15 (A5); no longer M5.14 (A6)
- net Shared_Address_A7: now also M5.16 (A4); no longer M5.13 (A7)
- net Shared_Address_A8: now also M5.1 (A11); no longer M5.3 (A8)
- net HSyncVGA renamed HSyncVGA_SuppressRCA
- net SYNC_RCA renamed VSyncVGA_RCA
Changed lines of the file:
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@@
 		)
 	)
-	(wire
-		(pts
-			(xy 601.98 429.26) (xy 598.17 429.26)
-		)
-		(stroke
-			(width 0)
-			(type default)
-		)
-	)
 	(bus
 		(pts
@@
 	(wire
 		(pts
-			(xy 551.18 355.6) (xy 591.82 355.6)
-		)
-		(stroke
-			(width 0)
-			(type default)
-		)
-	)
-	(wire
-		(pts
 			(xy 593.09 54.61) (xy 621.03 54.61)
 		)
@@
 	(wire
 		(pts
-			(xy 596.9 355.6) (xy 604.52 355.6)
-		)
-		(stroke
-			(width 0)
-			(type default)
-		)
-	)
-	(wire
-		(pts
 			(xy 195.58 444.5) (xy 175.26 444.5)
 		)
@@
 	(wire
 		(pts
-			(xy 551.18 429.26) (xy 593.09 429.26)
+			(xy 551.18 429.26) (xy 577.85 429.26)
 		)
 		(stroke
@@
 	(wire
 		(pts
+			(xy 551.18 355.6) (xy 577.85 355.6)
+		)
+		(stroke
+			(width 0)
+			(type default)
+		)
+	)
+	(wire
+		(pts
 			(xy 680.72 349.25) (xy 739.14 349.25)
 		)
@@
 		)
 	)
-	(label "Shared_Address_A7"
+	(label "Shared_Address_A4"
 		(at 332.74 431.8 180)
 		(effects
@@
 		)
 	)
-	(label "Shared_Address_A13"
+	(label "Shared_Address_A11"
 		(at 334.01 447.04 180)
 		(effects
@@
 		)
 	)
-	(label "Shared_Address_A14"
+	(label "Shared_Address_A13"
 		(at 334.01 449.58 180)
 		(effects
@@
 		)
 	)
-	(label "Shared_Address_A12"
+	(label "Shared_Address_A14"
 		(at 334.01 444.5 180)
 		(effects
@@
 		)
 	)
-	(label "Shared_Address_A11"
+	(label "Shared_Address_A8"
 		(at 334.01 441.96 180)
 		(effects
@@
 		)
 	)
-	(label "Shared_Address_A6"
+	(label "Shared_Address_A5"
 		(at 332.74 429.26 180)
 		(effects
@@
 		)
 	)
-	(label "Shared_Address_A10"
+	(label "Shared_Address_A15"
 		(at 334.01 439.42 180)
 		(effects
@@
 		)
 	)
-	(label "Shared_Address_A15"
+	(label "Shared_Address_A12"
 		(at 334.01 452.12 180)
 		(effects
@@
 		)
 	)
-	(label "Shared_Address_A8"
+	(label "Shared_Address_A10"
 		(at 332.74 434.34 180)
 		(effects
@@
 		)
 	)
-	(label "Shared_Address_A5"
+	(label "Shared_Address_A6"
 		(at 332.74 426.72 180)
 		(effects
@@
 		)
 	)
-	(label "Shared_Address_A4"
+	(label "Shared_Address_A7"
 		(at 332.74 424.18 180)
 		(effects
@@
 		)
 	)
-	(global_label "VSyncVGA"
+	(global_label "VSyncVGA_RCA"
 		(shape input)
 		(at 577.85 429.26 0)
@@
 		)
 	)
-	(global_label "~{SUPRESS}"
-		(shape input)
-		(at 604.52 355.6 0)
-		(fields_autoplaced yes)
-		(effects
-			(font
-				(size 1.27 1.27)
-			)
-			(justify left)
-		)
-		(property "Intersheetrefs" "${INTERSHEET_REFS}"
-			(at 616.1532 355.6 0)
-			(effects
-				(font
-					(size 1.27 1.27)
-				)
-				(justify left)
-				(hide yes)
-			)
-		)
-	)
 	(global_label "X_SHARE_DIRTY"
 		(shape input)
@@
 		)
 	)
-	(global_label "SYNC_RCA"
+	(global_label "VSyncVGA_RCA"
 		(shape input)
 		(at 506.73 623.57 180)
@@
 		)
 	)
-	(global_label "HSyncVGA"
+	(global_label "HSyncVGA_SuppressRCA"
 		(shape input)
 		(at 599.44 728.98 0)
@@
 		)
 	)
-	(global_label "VSyncVGA"
+	(global_label "VSyncVGA_RCA"
 		(shape input)
 		(at 600.71 734.06 0)
@@
 		)
 	)
-	(global_label "~{SUPRESS}"
+	(global_label "HSyncVGA_SuppressRCA"
 		(shape input)
 		(at 505.46 604.52 180)
@@
 		)
 	)
-	(global_label "HSyncVGA"
+	(global_label "HSyncVGA_SuppressRCA"
 		(shape input)
 		(at 577.85 355.6 0)
@@
 		)
 	)
-	(global_label "SYNC_RCA"
-		(shape input)
-		(at 601.98 429.26 0)
-		(fields_autoplaced yes)
-		(effects
-			(font
-				(size 1.27 1.27)
-			)
-			(justify left)
-		)
-		(property "Intersheetrefs" "${INTERSHEET_REFS}"
-			(at 614.46 429.26 0)
-			(effects
-				(font
-					(size 1.27 1.27)
-				)
-				(justify left)
-				(hide yes)
-			)
-		)
-	)
 	(global_label "X_HALT"
 		(shape input)
@@
 	)
 	(symbol
-		(lib_id "MHF:NetTie_2")
-		(at 594.36 355.6 0)
-		(mirror y)
-		(unit 1)
-		(exclude_from_sim no)
-		(in_bom no)
-		(on_board yes)
-		(dnp no)
-		(fields_autoplaced yes)
-		(property "Reference" "N3"
-			(at 594.36 353.314 0)
-			(effects
-				(font
-					(size 1.27 1.27)
-				)
-				(hide yes)
-			)
-		)
-		(property "Value" "~"
-			(at 594.36 351.79 0)
-			(effects
-				(font
-					(size 1.27 1.27)
-				)
-				(hide yes)
-			)
-		)
-		(property "Footprint" "MHF:NetTie-2_SMD_Pad0.5mm"
-			(at 594.36 355.6 0)
-			(effects
-				(font
-					(size 1.27 1.27)
-				)
-				(hide yes)
-			)
-		)
-		(property "Datasheet" "~"
-			(at 594.36 355.6 0)
-			(effects
-				(font
-					(size 1.27 1.27)
-				)
-				(hide yes)
-			)
-		)
-		(property "Description" "Net tie, 2 pins"
-			(at 594.36 355.6 0)
-			(effects
-				(font
-					(size 1.27 1.27)
-				)
-				(hide yes)
-			)
-		)
-		(pin "2"
-		)
-		(pin "1"
-		)
-		(instances
-			(project "MHF-002"
-				(path "/64851a36-d60f-4ef2-a652-2faeae5c6012"
-					(reference "N3")
-					(unit 1)
-				)
-			)
-		)
-	)
-	(symbol
 		(lib_id "MHF:R")
 		(at 544.83 601.98 90)
@@
 					(unit 1)
 				)
-			)
-		)
-	)
-	(symbol
-		(lib_id "MHF:NetTie_2")
-		(at 595.63 429.26 0)
-		(mirror y)
-		(unit 1)
-		(exclude_from_sim no)
-		(in_bom no)
-		(on_board yes)
-		(dnp no)
-		(fields_autoplaced yes)
-		(property "Reference" "N1"
-			(at 595.63 426.974 0)
-			(effects
-				(font
-					(size 1.27 1.27)
-				)
-				(hide yes)
-			)
-		)
-		(property "Value" "~"
-			(at 595.63 425.45 0)
-			(effects
-				(font
-					(size 1.27 1.27)
-				)
-				(hide yes)
-			)
-		)
-		(property "Footprint" "MHF:NetTie-2_SMD_Pad0.5mm"
-			(at 595.63 429.26 0)
-			(effects
-				(font
-					(size 1.27 1.27)
-				)
-				(hide yes)
-			)
-		)
-		(property "Datasheet" "~"
-			(at 595.63 429.26 0)
-			(effects
-				(font
-					(size 1.27 1.27)
-				)
-				(hide yes)
-			)
-		)
-		(property "Description" "Net tie, 2 pins"
-			(at 595.63 429.26 0)
-			(effects
-				(font
-					(size 1.27 1.27)
-				)
-				(hide yes)
-			)
-		)
-		(pin "2"
-		)
-		(pin "1"
-		)
-		(instances
-			(project "MHF-002"
-				(path "/64851a36-d60f-4ef2-a652-2faeae5c6012"
-					(reference "N1")
-					(unit 1)
-				)

Commit message: Silkscreen, views
Parts:
- added JP38: SHSelect, MHF:SolderJumper-3_P1.3mm_Open_RoundedPad1.0x1.5mm, symbol MHF:SolderJumper_3_Open
- added R50: 0?, MHF:R_0805_2012Metric_Pad1.20x1.40mm_HandSolder, symbol MHF:R
- JP102: value S_Enable -> S_SELECT
- JP35: value SBC_S_Enable -> SBC_S_SELECT
Connections:
- net +5V: now also R50.1; no longer U10.20 (VCC)
- net X_SHARE_DIRTY: now also JP34.1 (A); no longer JP35.1 (A)
- net A_SHARE_SELECT: now reaches J6.51 (Pin_51)
- net A_SHARE_SELECT: now also J4.51 (Pin_51), JP38.1 (A)
- net B_SHARE_SELECT: now reaches J6.52 (Pin_52)
- net B_SHARE_SELECT: now also J4.52 (Pin_52), JP38.3 (B)
- net A16 renamed A_16
- net A_S_ENABLE renamed A_S_SELECT
- net B16 renamed B_16
- net B_S_ENABLE renamed B_S_SELECT
- net S_ENABLE renamed S_SELECT
- net X_SHARE_FUTURE renamed X_SHARE_SELECT
- net X_SHARE_SELECT: now also JP35.1 (A), JP38.2 (C); no longer JP34.1 (A)
- new net: R50.2, U10.20 (VCC)
- no-connect marks 124 -> 120
Other:
- note added: "10-20 Ohm, or diode for restricting voltage and lowering ViH under 3.4V"
